File: PCB/ToolManger/ToolManger-15ports-schematic.sch (EAGLE design)
At the start: 52 parts, among them IC3 4049N, IC4 4049N, IC5 4049N

Commit message: UPDATE: board prototype finished
Connections:
- new net +5V: ESP_LEFT.15, JP4.1
- net GND: now also ESP_LEFT.14, JP1.10
Changed lines of the file:
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@@
 <class number="0" name="default" width="0" drill="0">
 </class>
-<class number="1" name="Supply" width="0.3" drill="0.8">
+<class number="1" name="Supply" width="0.5" drill="0.8">
 <clearance class="1" value="0.3"/>
 </class>
@@
 <part name="IC4" library="40xx" library_urn="urn:adsk.eagle:library:80" deviceset="4049" device="N" package3d_urn="urn:adsk.eagle:package:922/2"/>
 <part name="IC5" library="40xx" library_urn="urn:adsk.eagle:library:80" deviceset="4049" device="N" package3d_urn="urn:adsk.eagle:package:922/2"/>
+<part name="GND6" library="supply1" library_urn="urn:adsk.eagle:library:371" deviceset="GND" device=""/>
+<part name="P+1" library="supply1" library_urn="urn:adsk.eagle:library:371" deviceset="+5V" device=""/>
+<part name="P+2" library="supply1" library_urn="urn:adsk.eagle:library:371" deviceset="+5V" device=""/>
+<part name="GND7" library="supply1" library_urn="urn:adsk.eagle:library:371" deviceset="GND" device=""/>
 </parts>
 <sheets>
@@
 <instance part="IC3" gate="P" x="66.04" y="68.58" smashed="yes">
 <attribute name="NAME" x="64.77" y="67.945" size="1.778" layer="95"/>
+</instance>
+<instance part="GND6" gate="1" x="27.94" y="121.92" smashed="yes" rot="R270">
+<attribute name="VALUE" x="25.4" y="124.46" size="1.778" layer="96" rot="R270"/>
+</instance>
+<instance part="P+1" gate="1" x="22.86" y="111.76" smashed="yes" rot="R90">
+<attribute name="VALUE" x="27.94" y="109.22" size="1.778" layer="96" rot="R180"/>
+</instance>
+<instance part="P+2" gate="1" x="22.86" y="5.08" smashed="yes" rot="R90">
+<attribute name="VALUE" x="25.4" y="2.54" size="1.778" layer="96" rot="R180"/>
+</instance>
+<instance part="GND7" gate="1" x="22.86" y="7.62" smashed="yes" rot="R270">
+<attribute name="VALUE" x="20.32" y="10.16" size="1.778" layer="96" rot="R270"/>
 </instance>
 </instances>
@@
 <pinref part="IC5" gate="P" pin="VSS"/>
 </segment>
+<segment>
+<pinref part="GND6" gate="1" pin="GND"/>
+<pinref part="JP1" gate="A" pin="10"/>
+<wire x1="30.48" y1="121.92" x2="38.1" y2="121.92" width="0.1524" layer="91"/>
+</segment>
+<segment>
+<pinref part="GND7" gate="1" pin="GND"/>
+<pinref part="ESP_LEFT" gate="A" pin="14"/>
+<wire x1="25.4" y1="7.62" x2="30.48" y2="7.62" width="0.1524" layer="91"/>
+</segment>
 </net>
 <net name="+3V3" class="1">
@@
 </segment>
 </net>
+<net name="+5V" class="1">
+<segment>
+<pinref part="P+2" gate="1" pin="+5V"/>
+<pinref part="ESP_LEFT" gate="A" pin="15"/>
+<wire x1="25.4" y1="5.08" x2="30.48" y2="5.08" width="0.1524" layer="91"/>
+</segment>
+<segment>
+<pinref part="P+1" gate="1" pin="+5V"/>
+<pinref part="JP4" gate="A" pin="1"/>
+<wire x1="25.4" y1="111.76" x2="38.1" y2="111.76" width="0.1524" layer="91"/>
+</segment>
+</net>
